File: 4 Key Plate/Little_Big_Scroll_4KEY.sch (KiCad schematic (older format))
At the start: 9 parts, among them SW1 SW_Push, SW2 SW_Push, SW3 SW_Push, SW4 SW_Push, SW7 Rotary_Encoder_Switch

Commit message: folders
Parts:
- added Lic1: CC-BY-SA_4.0, Keyboard Library:CC_BY_SA_40, symbol Keyboard_Library:CC-BY-SA_4.0
Changed lines of the file:
@@
 Comp "Markus Knutsson <markus.knutsson@tweety.se>"
 Comment1 "https://github.com/TweetyDaBird"
-Comment2 "Licensed under CERN-OHL-S v2 or superseding version"
+Comment2 "Licensed under Creative Commons Attribution-ShareAlike 4.0 International"
 Comment3 ""
 Comment4 ""
@@
 	1    0    0    -1
 $EndComp
+$Comp
+L Keyboard_Library:CC-BY-SA_4.0 Lic1
+U 1 1 61A8B584
+P 8850 5500
+F 0 "Lic1" H 8850 5765 50  0000 C CNN
+F 1 "CC-BY-SA_4.0" H 8850 5674 50  0000 C CNN
+F 2 "Keyboard Library:CC_BY_SA_40" H 8850 5500 50  0001 C CNN
+F 3 "" H 8850 5500 50  0001 C CNN
+	1    8850 5500
+	1    0    0    -1
+$EndComp
