File: OLED Plate/Little_Big_Scroll_OLED.kicad_pcb (KiCad board)
At the start: 2 copper layers, 83.6 x 40 mm, 8 parts, among them SW3 SW_Push, SW4 SW_Push, SW7 Rotary_Encoder_Switch

Commit message: folders
Parts:
- added Lic1: CC-BY-SA_4.0, Keyboard Library:CC_BY_SA_40, B.Cu at (233.0, 112.3)
Other:
- board text added: "JLCJLCJLCJLC"
- board text added: "Little Big Scroll v1.0 Markus Knutsson 2021 https://github.com/TweetyDaBird"
- board text removed: "Little Big Scroll v1.0 Markus Knutsson 2021 https://github.com/TweetyDaBird Licensed under CERN-OHL-S v2+ JLCJLCJLCJLC"
