File: PCB/Little_Big_Scroll.sch (KiCad schematic (older format))
At the start: 22 parts, among them J1 Conn_01x02, SW1 SW_Push, SW2 SW_Push, SW3 SW_Push, SW4 SW_Push, SW7 Rotary_Encoder_Switch, U1 ProMicro

Commit message: folders
Parts:
- added Lic1: CC-BY-SA_4.0, Keyboard Library:CC_BY_SA_40, symbol Keyboard_Library:CC-BY-SA_4.0
Changed lines of the file:
@@
 Comp "Markus Knutsson <markus.knutsson@tweety.se>"
 Comment1 "https://github.com/TweetyDaBird"
-Comment2 "Licensed under CERN-OHL-S v2 or superseding version"
+Comment2 "Licensed under Creative Commons Attribution-ShareAlike 4.0 International"
 Comment3 ""
 Comment4 ""
@@
 Wire Wire Line
 	3550 1950 3200 1950
+$Comp
+L Keyboard_Library:CC-BY-SA_4.0 Lic1
+U 1 1 61A8D2CA
+P 9950 5950
+F 0 "Lic1" H 9950 6215 50  0000 C CNN
+F 1 "CC-BY-SA_4.0" H 9950 6124 50  0000 C CNN
+F 2 "Keyboard Library:CC_BY_SA_40" H 9950 5950 50  0001 C CNN
+F 3 "" H 9950 5950 50  0001 C CNN
+	1    9950 5950
+	1    0    0    -1
+$EndComp
 $EndSCHEMATC

Commit message: Tweaked for v1.1
Parts:
- R1, R2: footprint Resistor_THT:R_Axial_DIN0204_L3.6mm_D1.6mm_P5.08mm_Horizontal -> Resistor_THT:R_Axial_DIN0207_L6.3mm_D2.5mm_P7.62mm_Horizontal
- SW5: renamed from SW7; footprint Keebio-Parts:RotaryEncoder_Alps_EC11E-Switch_Vertical_H20mm -> Keyboard Library:RotaryEncoder_Alps_EC11E-Switch_Vertical_H20mm
Changed lines of the file:
@@
 $EndComp
 $Comp
-L Keyboard_Library:Rotary_Encoder_Switch_GND SW7
+L Keyboard_Library:Rotary_Encoder_Switch_GND SW5
 U 1 1 61F0CC2E
 P 8850 2050
-F 0 "SW7" H 8850 2417 50  0000 C CNN
+F 0 "SW5" H 8850 2417 50  0000 C CNN
 F 1 "Rotary_Encoder_Switch" H 8850 2326 50  0000 C CNN
-F 2 "Keebio-Parts:RotaryEncoder_Alps_EC11E-Switch_Vertical_H20mm" H 8700 2210 50  0001 C CNN
+F 2 "Keyboard Library:RotaryEncoder_Alps_EC11E-Switch_Vertical_H20mm" H 8700 2210 50  0001 C CNN
 F 3 "~" H 8850 2310 50  0001 C CNN
 	1    8850 2050
@@
 F 0 "R2" H 2050 4350 50  0000 R CNN
 F 1 "4K7" H 2100 4250 50  0000 R CNN
-F 2 "Resistor_THT:R_Axial_DIN0204_L3.6mm_D1.6mm_P5.08mm_Horizontal" H 1900 4300 50  0001 C CNN
+F 2 "Resistor_THT:R_Axial_DIN0207_L6.3mm_D2.5mm_P7.62mm_Horizontal" H 1900 4300 50  0001 C CNN
 F 3 "~" H 1900 4300 50  0001 C CNN
 	1    1900 4300
@@
 F 0 "R1" H 2109 4346 50  0000 L CNN
 F 1 "4K7" H 2109 4255 50  0000 L CNN
-F 2 "Resistor_THT:R_Axial_DIN0204_L3.6mm_D1.6mm_P5.08mm_Horizontal" H 2050 4300 50  0001 C CNN
+F 2 "Resistor_THT:R_Axial_DIN0207_L6.3mm_D2.5mm_P7.62mm_Horizontal" H 2050 4300 50  0001 C CNN
 F 3 "~" H 2050 4300 50  0001 C CNN
 	1    2050 4300
