File: Plate OLED/Little_Big_Scroll_OLED.kicad_pcb (KiCad board)
At the start: 2 copper layers, 83.6 x 40 mm, 9 parts, among them SW3 SW_Push, SW4 SW_Push, SW7 Rotary_Encoder_Switch

Commit message: Tweaked for v1.1
Parts:
- SW3, SW4: footprint keyswitches:Cherry_MX_Plate_Placeholder -> Keyboard Library:Cherry_MX_Plate_Placeholder
- SW7: footprint keyswitches:RotaryEncoder_PlateHole_Placeholder -> Keyboard Library:RotaryEncoder_PlateHole_Breakoff
Routing:
- removed copper zone on B.Cu, net (none)
- removed copper zone on F.Cu, net (none)
Other:
- board text added: "Little Big Scroll v1.1 Markus Knutsson 2022 https://github.com/TweetyDaBird"
- board text removed: "Little Big Scroll v1.0 Markus Knutsson 2021 https://github.com/TweetyDaBird"
