File: Plate OLED/Little_Big_Scroll_OLED.sch (KiCad schematic (older format))
At the start: 9 parts, among them SW3 SW_Push, SW4 SW_Push, SW7 Rotary_Encoder_Switch

Commit message: Tweaked for v1.1
Parts:
- SW3, SW4: footprint keyswitches:Cherry_MX_Plate_Placeholder -> Keyboard Library:Cherry_MX_Plate_Placeholder
- SW7: footprint keyswitches:RotaryEncoder_PlateHole_Placeholder -> Keyboard Library:RotaryEncoder_PlateHole_Breakoff
Connections:
- no-connect marks 0 -> 4
Changed lines of the file:
@@
 F 0 "SW3" H 5850 2535 50  0000 C CNN
 F 1 "SW_Push" H 5850 2444 50  0000 C CNN
-F 2 "keyswitches:Cherry_MX_Plate_Placeholder" H 5850 2450 50  0001 C CNN
+F 2 "Keyboard Library:Cherry_MX_Plate_Placeholder" H 5850 2450 50  0001 C CNN
 F 3 "~" H 5850 2450 50  0001 C CNN
 	1    5850 2250
@@
 F 0 "SW4" H 6250 2885 50  0000 C CNN
 F 1 "SW_Push" H 6250 2794 50  0000 C CNN
-F 2 "keyswitches:Cherry_MX_Plate_Placeholder" H 6250 2800 50  0001 C CNN
+F 2 "Keyboard Library:Cherry_MX_Plate_Placeholder" H 6250 2800 50  0001 C CNN
 F 3 "~" H 6250 2800 50  0001 C CNN
 	1    6250 2600
@@
 F 0 "SW7" H 8850 2417 50  0000 C CNN
 F 1 "Rotary_Encoder_Switch" H 8850 2326 50  0000 C CNN
-F 2 "keyswitches:RotaryEncoder_PlateHole_Placeholder" H 8700 2210 50  0001 C CNN
+F 2 "Keyboard Library:RotaryEncoder_PlateHole_Breakoff" H 8700 2210 50  0001 C CNN
 F 3 "~" H 8850 2310 50  0001 C CNN
 	1    8850 2050
@@
 	1    0    0    -1
 $EndComp
+NoConn ~ 2500 4000
+NoConn ~ 2500 4100
+NoConn ~ 2500 4200
+NoConn ~ 2500 4300
 $EndSCHEMATC
