File: Little Big Scroll 4/PCB/Little_Big_Scroll_4.sch (KiCad schematic (older format))
At the start: 23 parts, among them J1 Conn_01x02, SW1 SW_Push, SW2 SW_Push, SW3 SW_Push, SW4 SW_Push, SW5 Rotary_Encoder_Switch, U1 ProMicro

Commit message: Renamed to 'Little Big Scroll 4'
Parts:
- added D1, D2, D3, D4, D5: 1N4148, Diode_THT:D_DO-35_SOD27_P7.62mm_Horizontal, symbol Diode:1N4148
Connections:
- net ROW3 is gone; now on net COL1: SW4.1, U1.10 (E6)
- net ROW4 is gone; now on net COL3: SW5.S2, U1.20 ((A)F4)
- net COL0: now also SW1.1, SW3.1; no longer SW1.2
- net COL1: now also SW2.1; no longer SW2.2, U1.8 (C6)
- net COL3: no longer SW4.2, U1.11 (B4)
- net ROW0: now also U1.11 (B4), D1.1 (K), D2.1 (K), D5.1 (K); no longer SW1.1, U1.1 (D3(TX))
- net ROW1: now also U1.12 (B5), D3.1 (K), D4.1 (K); no longer SW2.1, U1.7 (D4)
- net COL2: no longer names the net of SW3.2
- net COL2: now also D3.2 (A); no longer U1.13 (B6)
- net COL4: no longer names the net of SW5.S1
- net COL4: now also D5.2 (A); no longer U1.19 ((A)F5)
- removed net ROW2: SW3.1, U1.12 (B5)
- new net: D1.2 (A), SW1.2
- new net: D2.2 (A), SW2.2
- new net: D4.2 (A), SW4.2
- no-connect marks 5 -> 2
Other:
- moved on the sheet: SW1, SW2, SW3, SW4
Changed lines of the file:
@@
 $EndComp
 NoConn ~ 3200 1850
-NoConn ~ 3200 2850
-Text GLabel 1800 1950 0    50   Output ~ 0
-RGB
 $Comp
 L power:GND #PWR0101
@@
 L Switch:SW_Push SW1
 U 1 1 61F07A41
-P 5050 1550
-F 0 "SW1" H 5050 1835 50  0000 C CNN
-F 1 "SW_Push" H 5050 1744 50  0000 C CNN
-F 2 "keyswitches:Kailh_socket_MX_RGB" H 5050 1750 50  0001 C CNN
-F 3 "~" H 5050 1750 50  0001 C CNN
-	1    5050 1550
-	1    0    0    -1
+P 5050 1350
+F 0 "SW1" H 5050 1635 50  0000 C CNN
+F 1 "SW_Push" H 5050 1544 50  0000 C CNN
+F 2 "keyswitches:Kailh_socket_MX_RGB" H 5050 1550 50  0001 C CNN
+F 3 "~" H 5050 1550 50  0001 C CNN
+	1    5050 1350
+	-1   0    0    -1
 $EndComp
 $Comp
 L Switch:SW_Push SW2
 U 1 1 61F08A46
-P 5450 1900
-F 0 "SW2" H 5450 2185 50  0000 C CNN
-F 1 "SW_Push" H 5450 2094 50  0000 C CNN
-F 2 "keyswitches:Kailh_socket_MX_RGB" H 5450 2100 50  0001 C CNN
-F 3 "~" H 5450 2100 50  0001 C CNN
-	1    5450 1900
-	1    0    0    -1
+P 5600 1350
+F 0 "SW2" H 5600 1635 50  0000 C CNN
+F 1 "SW_Push" H 5600 1544 50  0000 C CNN
+F 2 "keyswitches:Kailh_socket_MX_RGB" H 5600 1550 50  0001 C CNN
+F 3 "~" H 5600 1550 50  0001 C CNN
+	1    5600 1350
+	-1   0    0    -1
 $EndComp
 $Comp
 L Switch:SW_Push SW3
 U 1 1 61F08FF4
-P 5850 2250
-F 0 "SW3" H 5850 2535 50  0000 C CNN
-F 1 "SW_Push" H 5850 2444 50  0000 C CNN
-F 2 "keyswitches:Kailh_socket_MX_RGB" H 5850 2450 50  0001 C CNN
-F 3 "~" H 5850 2450 50  0001 C CNN
-	1    5850 2250
-	1    0    0    -1
+P 5050 2050
+F 0 "SW3" H 5050 2335 50  0000 C CNN
+F 1 "SW_Push" H 5050 2244 50  0000 C CNN
+F 2 "keyswitches:Kailh_socket_MX_RGB" H 5050 2250 50  0001 C CNN
+F 3 "~" H 5050 2250 50  0001 C CNN
+	1    5050 2050
+	-1   0    0    -1
 $EndComp
 $Comp
 L Switch:SW_Push SW4
 U 1 1 61F0A1A5
-P 6250 2600
-F 0 "SW4" H 6250 2885 50  0000 C CNN
-F 1 "SW_Push" H 6250 2794 50  0000 C CNN
-F 2 "keyswitches:Kailh_socket_MX_RGB" H 6250 2800 50  0001 C CNN
-F 3 "~" H 6250 2800 50  0001 C CNN
-	1    6250 2600
-	1    0    0    -1
+P 5600 2050
+F 0 "SW4" H 5600 2335 50  0000 C CNN
+F 1 "SW_Push" H 5600 2244 50  0000 C CNN
+F 2 "keyswitches:Kailh_socket_MX_RGB" H 5600 2250 50  0001 C CNN
+F 3 "~" H 5600 2250 50  0001 C CNN
+	1    5600 2050
+	-1   0    0    -1
 $EndComp
 $Comp
@@
 	7900 2250 8100 2250
 Connection ~ 8100 2250
-Text GLabel 3200 2650 2    50   Input ~ 0
-ENC_A
-Text GLabel 3200 2550 2    50   Input ~ 0
-ENC_B
 $Comp
 L Device:R_Small R2
@@
 	1    0    0    -1
 $EndComp
-Text GLabel 5250 1100 0    50   Input ~ 0
+Text GLabel 5250 900  0    50   Input ~ 0
 COL0
-Text GLabel 5650 1100 0    50   Input ~ 0
+Text GLabel 5800 900  0    50   Input ~ 0
 COL1
-Text GLabel 6050 1100 0    50   Input ~ 0
-COL2
-Text GLabel 6450 1100 0    50   Input ~ 0
-COL3
-Text GLabel 4850 1550 0    50   Input ~ 0
+Text GLabel 4750 1650 0    50   Input ~ 0
 ROW0
-Text GLabel 4850 1900 0    50   Input ~ 0
+Text GLabel 4750 2350 0    50   Input ~ 0
 ROW1
-Text GLabel 4850 2250 0    50   Input ~ 0
-ROW2
-Text GLabel 4850 2600 0    50   Input ~ 0
-ROW3
-Wire Wire Line
-	5250 1900 4850 1900
-Wire Wire Line
-	5250 1100 5250 1550
-Wire Wire Line
-	5650 1900 5650 1100
-Wire Wire Line
-	4850 2250 5650 2250
-Wire Wire Line
-	6050 2250 6050 1100
-Wire Wire Line
-	6050 2600 4850 2600
-Wire Wire Line
-	6450 2600 6450 1100
-Text GLabel 9150 1950 2    50   Input ~ 0
-COL4
-Text GLabel 9150 2150 2    50   Input ~ 0
-ROW4
-Text GLabel 1800 1850 0    50   Input ~ 0
-ROW0
-Text GLabel 1800 2450 0    50   Input ~ 0
-ROW1
-Text GLabel 1800 2950 0    50   Input ~ 0
-ROW2
-Text GLabel 1800 2750 0    50   Input ~ 0
-ROW3
-Text GLabel 3200 2250 2    50   Input ~ 0
-ROW4
-Text GLabel 1800 2850 0    50   Input ~ 0
-COL3
-Text GLabel 3200 2950 2    50   Input ~ 0
-COL2
-Text GLabel 1800 2550 0    50   Input ~ 0
-COL1
-Text GLabel 1800 2650 0    50   Input ~ 0
-COL0
-Text GLabel 3200 2350 2    50   Input ~ 0
-COL4
-NoConn ~ 3200 2450
-NoConn ~ 3200 2750
+Wire Wire Line
+	5250 900  5250 1350
+Wire Wire Line
+	4750 2350 4850 2350
 $Comp
 L Connector_Generic:Conn_01x02 J1
@@
 	1    0    0    -1
 $EndComp
+Wire Wire Line
+	5800 1350 5800 900
+$Comp
+L Diode:1N4148 D1
+U 1 1 61E206D2
+P 4850 1500
+F 0 "D1" V 4896 1420 50  0000 R CNN
+F 1 "1N4148" V 4805 1420 50  0000 R CNN
+F 2 "Diode_THT:D_DO-35_SOD27_P7.62mm_Horizontal" H 4850 1325 50  0001 C CNN
+F 3 "https://assets.nexperia.com/documents/data-sheet/1N4148_1N4448.pdf" H 4850 1500 50  0001 C CNN
+	1    4850 1500
+	0    -1   -1   0
+$EndComp
+$Comp
+L Diode:1N4148 D2
+U 1 1 61E253A0
+P 5400 1500
+F 0 "D2" V 5446 1420 50  0000 R CNN
+F 1 "1N4148" V 5355 1420 50  0000 R CNN
+F 2 "Diode_THT:D_DO-35_SOD27_P7.62mm_Horizontal" H 5400 1325 50  0001 C CNN
+F 3 "https://assets.nexperia.com/documents/data-sheet/1N4148_1N4448.pdf" H 5400 1500 50  0001 C CNN
+	1    5400 1500
+	0    -1   -1   0
+$EndComp
+Wire Wire Line
+	4750 1650 4850 1650
+Connection ~ 4850 1650
+Wire Wire Line
+	4850 1650 5400 1650
+$Comp
+L Diode:1N4148 D3
+U 1 1 61E2B13C
+P 4850 2200
+F 0 "D3" V 4896 2120 50  0000 R CNN
+F 1 "1N4148" V 4805 2120 50  0000 R CNN
+F 2 "Diode_THT:D_DO-35_SOD27_P7.62mm_Horizontal" H 4850 2025 50  0001 C CNN
+F 3 "https://assets.nexperia.com/documents/data-sheet/1N4148_1N4448.pdf" H 4850 2200 50  0001 C CNN
+	1    4850 2200
+	0    -1   -1   0
+$EndComp
+$Comp
+L Diode:1N4148 D4
+U 1 1 61E2BE9C
+P 5400 2200
+F 0 "D4" V 5446 2120 50  0000 R CNN
+F 1 "1N4148" V 5355 2120 50  0000 R CNN
+F 2 "Diode_THT:D_DO-35_SOD27_P7.62mm_Horizontal" H 5400 2025 50  0001 C CNN
+F 3 "https://assets.nexperia.com/documents/data-sheet/1N4148_1N4448.pdf" H 5400 2200 50  0001 C CNN
+	1    5400 2200
+	0    -1   -1   0
+$EndComp
+Connection ~ 4850 2350
+Wire Wire Line
+	4850 2350 5400 2350
+Wire Wire Line
+	5250 1350 5250 2050
+Connection ~ 5250 1350
+Wire Wire Line
+	5800 1350 5800 2050
+Connection ~ 5800 1350
+Text GLabel 9450 1950 2    50   Input ~ 0
+ROW0
+Text GLabel 9450 2150 2    50   Input ~ 0
+COL3
+Text GLabel 1800 1950 0    50   Output ~ 0
+RGB
+$Comp
+L Diode:1N4148 D5
+U 1 1 61E57772
+P 9300 1950
+F 0 "D5" H 9300 2167 50  0000 C CNN
+F 1 "1N4148" H 9300 2076 50  0000 C CNN
+F 2 "Diode_THT:D_DO-35_SOD27_P7.62mm_Horizontal" H 9300 1775 50  0001 C CNN
+F 3 "https://assets.nexperia.com/documents/data-sheet/1N4148_1N4448.pdf" H 9300 1950 50  0001 C CNN
+	1    9300 1950
+	-1   0    0    -1
+$EndComp
+Wire Wire Line
+	9450 2150 9150 2150
+Text GLabel 1800 2850 0    50   Input ~ 0
+ROW0
+Text GLabel 1800 2950 0    50   Input ~ 0
+ROW1
+Text GLabel 1800 2650 0    50   Input ~ 0
+COL0
+Text GLabel 1800 2750 0    50   Input ~ 0
+COL1
+Text GLabel 3200 2250 2    50   Input ~ 0
+COL3
+Text GLabel 3200 2650 2    50   Input ~ 0
+ENC_A
+Text GLabel 3200 2550 2    50   Input ~ 0
+ENC_B
 $EndSCHEMATC

Commit message: Added Little Big Scroll 6
Parts:
- added H5: Hole, QMK Logo:Powered_by_QMK, symbol Keyboard_Library:Hole
Changed lines of the file:
@@
 encoding utf-8
 Sheet 1 1
-Title "Little Big Scroll"
-Date "2021-11-30"
-Rev "v1.0"
+Title "Little Big Scroll 4"
+Date "2022-01-10"
+Rev "v1.1"
 Comp "Markus Knutsson <markus.knutsson@tweety.se>"
 Comment1 "https://github.com/TweetyDaBird"
@@
 Text GLabel 3200 2550 2    50   Input ~ 0
 ENC_B
+$Comp
+L Keyboard_Library:Hole H5
+U 1 1 61E6F18C
+P 12750 2150
+F 0 "H5" H 12936 2203 60  0000 L CNN
+F 1 "Hole" H 12936 2097 60  0000 L CNN
+F 2 "QMK Logo:Powered_by_QMK" H 12750 2150 60  0001 C CNN
+F 3 "" H 12750 2150 60  0001 C CNN
+	1    12750 2150
+	1    0    0    -1
+$EndComp
 $EndSCHEMATC
