File: Little Big Scroll 4/PCB/Little_Big_Scroll_4.kicad_pcb (KiCad board)
At the start: 2 copper layers, 83.6 x 40 mm, 29 parts, among them J1 Conn_01x02, SW1 SW_Push, SW2 SW_Push, SW3 SW_Push, SW4 SW_Push, SW5 Rotary_Encoder_Switch, U1 ProMicro

Commit message: Added Little Big Scroll 6
Parts:
- removed D1, D2, D3, D4, D5: 1N4148, Diode_THT:D_DO-35_SOD27_P7.62mm_Horizontal
- Logo1: renamed from H5; value Hole -> QMK_Logo
Connections:
- LED6 pad 2: (no net) -> unconnected-(LED6-Pad2)
- SW1 pad 1: COL0 -> GND
- SW1 pad 2: Net-(D1-Pad2) -> Key1
- SW2 pad 1: COL1 -> GND
- SW2 pad 2: Net-(D2-Pad2) -> Key2
- SW3 pad 1: COL0 -> GND
- SW3 pad 2: Net-(D3-Pad2) -> Key3
- SW4 pad 1: COL1 -> GND
- SW4 pad 2: Net-(D4-Pad2) -> Key4
- SW5 pad S1: Net-(D5-Pad2) -> Key5
- SW5 pad S2: COL3 -> GND
- U1 pad 1: (no net) -> unconnected-(U1-Pad1)
- U1 pad 10: COL1 -> Key1
- U1 pad 11: ROW0 -> Key4
- U1 pad 12: ROW1 -> Key3
- U1 pad 13: (no net) -> unconnected-(U1-Pad13)
- U1 pad 14: (no net) -> unconnected-(U1-Pad14)
- U1 pad 15: (no net) -> unconnected-(U1-Pad15)
- U1 pad 18: (no net) -> unconnected-(U1-Pad18)
- U1 pad 19: (no net) -> unconnected-(U1-Pad19)
- U1 pad 20: COL3 -> Key5
- U1 pad 24: (no net) -> unconnected-(U1-Pad24)
- U1 pad 7: (no net) -> unconnected-(U1-Pad7)
- U1 pad 8: (no net) -> unconnected-(U1-Pad8)
- U1 pad 9: COL0 -> Key2
Routing:
- net ROW0: track 117.7 -> 0.00 mm
- net Key1: track 0.00 -> 52.2 mm, vias 0 -> 1
- net COL0: track 46.4 -> 0.00 mm, vias 2 -> 0
- net Key3: track 0.00 -> 41.2 mm, vias 0 -> 1
- net ROW1: track 39.7 -> 0.00 mm
- net VCC: track 188.3 -> 149.9 mm, vias 4 -> 7
- net Key2: track 0.00 -> 33.4 mm, vias 0 -> 2
- net COL1: track 27.6 -> 0.00 mm, vias 2 -> 0
- net Key4: track 0.00 -> 22.7 mm, vias 0 -> 1
- net Key5: track 0.00 -> 11.3 mm
- net Net-(D4-Pad2): track 9.73 -> 0.00 mm, vias 1 -> 0
- net Net-(LED5-Pad2): track 29.7 -> 37.8 mm, vias 0 -> 2
- net Net-(D2-Pad2): track 7.26 -> 0.00 mm, vias 1 -> 0
- net Net-(D1-Pad2): track 7.16 -> 0.00 mm, vias 1 -> 0
- net Net-(D3-Pad2): track 6.35 -> 0.00 mm, vias 1 -> 0
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Other:
- net class Default removed
- net class VCC removed
- board text added: "Little Big Scroll 4 v1.11 Markus Knutsson 2022 https://github.com/TweetyDaBird"
- board text removed: "Little Big Scroll 4 v1.1 Markus Knutsson 2022 https://github.com/TweetyDaBird"
