File: Little Big Scroll 6/Front Plate/LBS6_Front_Plate.kicad_sch (KiCad schematic)
At the start: 13 parts, among them SW1 SW_Push, SW2 SW_Push, SW3 SW_Push, SW4 SW_Push, SW5 SW_Push, SW6 SW_Push, SW7 Rotary_Encoder_Switch

Commit message: LBS6 v1.01
Parts:
- H1, H2, H3, H4: footprint MountingHole:MountingHole_3.7mm -> Tweety keyswitches:Plate_Hole
- SW1, SW2, SW3, SW4, SW5, SW6: footprint Tweety keyswitches:Plate_1u -> Tweety keyswitches:Cherry_MX_Plate_Placeholder; symbol Keyswitches:SW_Push -> Switch:SW_Push
- SW7: footprint Keyboard Library:RotaryEncoder_PlateHole_Placeholder -> Tweety keyswitches:Plate_Encoder

Commit message: LSB6 1.01
Parts:
- ENC1: renamed from SW7; value Rotary_Encoder_Switch -> (none); footprint Tweety keyswitches:Plate_Encoder -> (none); symbol Keyboard_Library:Encoder_Switch_GND -> Keyboard Switches & Encoders:Rotary_Encoder_Click
- H1, H2, H3, H4: value Hole_PCB_M2-Spacer -> Spacer_Plate; footprint Tweety keyswitches:Plate_Hole -> Keyboard Switches & Encoders:Spacer Plate hole; symbol Keyboard_Library:Hole_PCB_M2-Spacer -> Keyboard Switches & Encoders:Spacer_Plate
- Logo1: renamed from Lic1; footprint CC_Licensing:CC_BY_SA_40 -> Logotypes:CC_BY_SA_40; symbol CC_Licensing:CC-BY-SA-4.0 -> Logotypes:CC-BY-SA-4.0
- Logo2: renamed from Logo1; footprint QMK Logo:Powered_by_QMK -> Logotypes:Powered_by_QMK; symbol Keyboard Library:QMK_Logo -> Logotypes:QMK_Logo; now left out of the parts list
- SW1, SW2, SW3, SW4, SW5, SW6: footprint Tweety keyswitches:Cherry_MX_Plate_Placeholder -> Keyboard Switches & Encoders:SW_MX_Plate_Placeholder
Other:
- moved on the sheet: Logo2
