File: Little Big Scroll 6/PCB/Little Big Scroll 6.kicad_sch (KiCad schematic)
At the start: 25 parts, among them J1 Conn_01x02, SW1 SW_Push, SW2 SW_Push, SW3 SW_Push, SW4 SW_Push, SW5 SW_Push, SW6 SW_Push, SW7 Rotary_Encoder_Switch, U1 ProMicro

Commit message: LBS6 v1.01
Parts:
- added J2: Conn_01x02, Connector_JST:JST_PH_S2B-PH-K_1x02_P2.00mm_Horizontal, symbol Connector_Generic:Conn_01x02
- added S1: MSK12C02, MSK12C02, symbol Keyboard Library:MSK12C02
Connections:
- net GND: now also J2.1 (Pin_1), S1.MP
- net BAT+: now reaches U1.24 (RAW)
- net BAT+: now also S1.B1 (COM)
- new net BAT++: J2.2 (Pin_2), S1.C1 (NO)
- no-connect marks 10 -> 9
Changed lines of the file:
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@@
   (title_block
     (title "Little Big Scroll 6")
-    (date "2022-01-28")
-    (rev "v1.0")
+    (date "2022-03-22")
+    (rev "v1.01")
     (company "Tweety's Wild Thinking")
     (comment 1 "Markus Knutsson <markus.knutsson@tweety.se>")
@@
   (no_connect (at 74.93 59.69))
   (no_connect (at 39.37 44.45))
-  (no_connect (at 74.93 34.29))
   (no_connect (at 39.37 34.29))
   (no_connect (at 74.93 44.45))
@@
     (stroke (width 0) (type default) (color 0 0 0 0))
   )
+  (wire (pts (xy 167.386 92.71) (xy 167.386 96.52))
+    (stroke (width 0) (type default) (color 0 0 0 0))
+  )
+  (wire (pts (xy 181.61 109.22) (xy 172.212 109.22))
+    (stroke (width 0) (type default) (color 0 0 0 0))
+  )
   (wire (pts (xy 53.34 107.95) (xy 43.18 107.95))
     (stroke (width 0) (type default) (color 0 0 0 0))
@@
     (stroke (width 0) (type default) (color 0 0 0 0))
   )
+  (wire (pts (xy 172.212 95.25) (xy 172.212 109.22))
+    (stroke (width 0) (type default) (color 0 0 0 0))
+  )
   (wire (pts (xy 167.64 29.21) (xy 167.64 49.53))
     (stroke (width 0) (type default) (color 0 0 0 0))
@@
     (stroke (width 0) (type default) (color 0 0 0 0))
   )
+  (wire (pts (xy 172.212 92.71) (xy 167.386 92.71))
+    (stroke (width 0) (type default) (color 0 0 0 0))
+  )
   (wire (pts (xy 168.91 44.45) (xy 179.07 44.45))
     (stroke (width 0) (type default) (color 0 0 0 0))
@@
   (wire (pts (xy 179.07 29.21) (xy 196.85 29.21))
     (stroke (width 0) (type default) (color 0 0 0 0))
+  )
+  (label "BAT++" (at 172.212 101.092 0)
+    (effects (font (size 1.27 1.27)) (justify left bottom))
   )
   (global_label "Key3" (shape input) (at 120.65 114.3 180) (fields_autoplaced)
@@
     )
   )
+  (global_label "BAT+" (shape input) (at 74.93 34.29 0) (fields_autoplaced)
+    (effects (font (size 1.27 1.27)) (justify left))
+    (property "Intersheet References" "${INTERSHEET_REFS}" (id 0) (at 82.1528 34.2106 0)
+      (effects (font (size 1.27 1.27)) (justify left) hide)
+    )
+  )
   (global_label "Key1" (shape input) (at 120.65 93.98 180) (fields_autoplaced)
     (effects (font (size 1.27 1.27)) (justify right))
@@
     (property "Intersheet References" "${INTERSHEET_REFS}" (id 0) (at -22.86 -20.32 0)
       (effects (font (size 1.27 1.27)) hide)
+    )
+  )
+  (global_label "BAT+" (shape input) (at 181.61 106.68 180) (fields_autoplaced)
+    (effects (font (size 1.27 1.27)) (justify right))
+    (property "Intersheet References" "${INTERSHEET_REFS}" (id 0) (at 174.3872 106.7594 0)
+      (effects (font (size 1.27 1.27)) (justify right) hide)
     )
   )
@@
     )
   )
+  (symbol (lib_id "power:GND") (at 190.5 114.3 0) (unit 1)
+    (in_bom yes) (on_board yes)
+    (property "Reference" "#PWR0113" (id 0) (at 190.5 120.65 0)
+      (effects (font (size 1.27 1.27)) hide)
+    )
+    (property "Value" "GND" (id 1) (at 190.627 118.6942 0))
+    (property "Footprint" "" (id 2) (at 190.5 114.3 0)
+      (effects (font (size 1.27 1.27)) hide)
+    )
+    (property "Datasheet" "" (id 3) (at 190.5 114.3 0)
+      (effects (font (size 1.27 1.27)) hide)
+    )
+    (pin "1")
+  )
   (symbol (lib_id "Connector_Generic:Conn_01x02") (at 99.06 41.91 0) (mirror x) (unit 1)
     (in_bom yes) (on_board yes) (fields_autoplaced)
@@
     (pin "1")
   )
+  (symbol (lib_id "Keyboard Library:MSK12C02") (at 189.23 107.95 0) (unit 1)
+    (in_bom yes) (on_board yes) (fields_autoplaced)
+    (property "Reference" "S1" (id 0) (at 196.2912 105.7715 0)
+      (effects (font (size 1.27 1.27)) (justify left))
+    )
+    (property "Value" "MSK12C02" (id 1) (at 196.2912 108.5466 0)
+      (effects (font (size 1.27 1.27)) (justify left))
+    )
+    (property "Footprint" "MSK12C02" (id 2) (at 199.39 101.6 0)
+      (effects (font (size 1.27 1.27)) (justify left) hide)
+    )
+    (property "Datasheet" "https://shouhan.en.made-in-china.com/product/xsMEmqgOAXWB/China-Slide-Switch-Msk12c02-Slide-Switch-on-off-2-Position-1p2t-Spdt-Miniature-Horizontal-SMD-7p-Slide-Switch.html" (id 3) (at 199.39 104.14 0)
+      (effects (font (size 1.27 1.27)) (justify left) hide)
+    )
+    (property "Description" "SMD Toggle Switches" (id 4) (at 199.39 106.68 0)
+      (effects (font (size 1.27 1.27)) (justify left) hide)
+    )
+    (property "Height" "1.4" (id 5) (at 199.39 109.22 0)
+      (effects (font (size 1.27 1.27)) (justify left) hide)
+    )
+    (property "Manufacturer_Name" "Shou Han" (id 6) (at 199.39 111.76 0)
+      (effects (font (size 1.27 1.27)) (justify left) hide)
+    )
+    (property "Manufacturer_Part_Number" "MSK12C02" (id 7) (at 199.39 114.3 0)
+      (effects (font (size 1.27 1.27)) (justify left) hide)
+    )
+    (pin "A1")
+    (pin "B1")
+    (pin "C1")
+    (pin "MP")
+  )
   (symbol (lib_id "power:GND") (at 160.02 186.69 0) (unit 1)
     (in_bom yes) (on_board yes)
@@
     )
     (property "Datasheet" "" (id 3) (at 168.91 186.69 0)
+      (effects (font (size 1.27 1.27)) hide)
+    )
+    (pin "1")
+  )
+  (symbol (lib_id "power:GND") (at 167.386 96.52 0) (unit 1)
+    (in_bom yes) (on_board yes)
+    (property "Reference" "#PWR0112" (id 0) (at 167.386 102.87 0)
+      (effects (font (size 1.27 1.27)) hide)
+    )
+    (property "Value" "GND" (id 1) (at 167.513 100.9142 0))
+    (property "Footprint" "" (id 2) (at 167.386 96.52 0)
+      (effects (font (size 1.27 1.27)) hide)
+    )
+    (property "Datasheet" "" (id 3) (at 167.386 96.52 0)
       (effects (font (size 1.27 1.27)) hide)
     )
@@
     (pin "1")
   )
+  (symbol (lib_id "Connector_Generic:Conn_01x02") (at 177.292 92.71 0) (unit 1)
+    (in_bom yes) (on_board yes) (fields_autoplaced)
+    (property "Reference" "J2" (id 0) (at 179.324 93.0715 0)
+      (effects (font (size 1.27 1.27)) (justify left))
+    )
+    (property "Value" "Conn_01x02" (id 1) (at 179.324 95.8466 0)
+      (effects (font (size 1.27 1.27)) (justify left))
+    )
+    (property "Footprint" "Connector_JST:JST_PH_S2B-PH-K_1x02_P2.00mm_Horizontal" (id 2) (at 177.292 92.71 0)
+      (effects (font (size 1.27 1.27)) hide)
+    )
+    (property "Datasheet" "~" (id 3) (at 177.292 92.71 0)
+      (effects (font (size 1.27 1.27)) hide)
+    )
+    (pin "1")
+    (pin "2")
+  )
   (sheet_instances
     (path "/" (page "1"))
@@
       (reference "#PWR0111") (unit 1) (value "GND") (footprint "")
     )
+    (path "/99c7eb7c-a47e-40e7-ace7-a2d71007b07e"
+      (reference "#PWR0112") (unit 1) (value "GND") (footprint "")
+    )
+    (path "/2b633fa8-851e-4eb1-8dd4-9842c9dcb9e1"
+      (reference "#PWR0113") (unit 1) (value "GND") (footprint "")
+    )
     (path "/00000000-0000-0000-0000-000061f8dbc6"
       (reference "C1") (unit 1) (value "100nF") (footprint "Capacitor_THT:C_Axial_L3.8mm_D2.6mm_P7.50mm_Horizontal")
@@
       (reference "J1") (unit 1) (value "Conn_01x02") (footprint "Connector_PinHeader_2.54mm:PinHeader_1x02_P2.54mm_Vertical")
     )
+    (path "/f2ef9832-cd91-4ae7-b753-a4bc69dff2eb"
+      (reference "J2") (unit 1) (value "Conn_01x02") (footprint "Connector_JST:JST_PH_S2B-PH-K_1x02_P2.00mm_Horizontal")
+    )
     (path "/00000000-0000-0000-0000-000061eeb947"
       (reference "LED1") (unit 1) (value "SK6812MINI-E") (footprint "kicad-keyboard-parts:MX_SK6812MINI-E")
@@
       (reference "Logo1") (unit 1) (value "QMK_Logo") (footprint "QMK Logo:Powered_by_QMK")
     )
+    (path "/7fc6eda3-a41a-4ab9-935d-37e18cb30594"
+      (reference "S1") (unit 1) (value "MSK12C02") (footprint "MSK12C02")
+    )
     (path "/00000000-0000-0000-0000-000061e9d956"

Commit message: LSB6 1.01
Parts:
- removed SW1, SW2, SW3, SW4, SW5, SW6: SW_Push, keyswitches:Kailh_socket_MX_RGB, symbol Switch:SW_Push
- added SW1, SW2, SW3, SW4, SW5, SW6: SW_MX_HS, Keyboard Switches & Encoders:SW_MX_HotSwap, symbol Keyboard Switches & Encoders:SW_MX_HS
- C1, C2: value 100nF -> C_Small; footprint Capacitor_THT:C_Axial_L3.8mm_D2.6mm_P7.50mm_Horizontal -> (none)
- ENC1: renamed from SW7; value Rotary_Encoder_Switch -> Rotary_Encoder_Click; footprint Keyboard Library:RotaryEncoder_Alps_EC11E-Switch_Vertical_H20mm -> Keyboard Switches & Encoders:Encoder_Alps_EC11E; symbol Keyboard_Library:Encoder_Switch_GND -> Keyboard Switches & Encoders:Rotary_Encoder_Click
- H1, H2, H3, H4: value Hole_PCB_M2-Spacer -> Spacer_PCB; footprint MountingHole:MountingHole_3.7mm -> Keyboard Switches & Encoders:Spacer PCB hole; symbol Keyboard_Library:Hole_PCB_M2-Spacer -> Keyboard Switches & Encoders:Spacer_PCB
- J1: footprint Connector_PinHeader_2.54mm:PinHeader_1x02_P2.54mm_Vertical -> (none)
- J2: footprint Connector_JST:JST_PH_S2B-PH-K_1x02_P2.00mm_Horizontal -> (none)
- Logo1: renamed from Lic1; footprint CC_Licensing:CC_BY_SA_40 -> Logotypes:CC_BY_SA_40; symbol CC_Licensing:CC-BY-SA-4.0 -> Logotypes:CC-BY-SA-4.0
- Logo2: renamed from Logo1; footprint QMK Logo:Powered_by_QMK -> Logotypes:Powered_by_QMK; symbol Keyboard Library:QMK_Logo -> Logotypes:QMK_Logo; now left out of the parts list
- RGB1: renamed from LED1; footprint kicad-keyboard-parts:MX_SK6812MINI-E -> Keyboard Switches & Encoders:RGB_SK6812MINI-E; symbol Keyboard_Library:SK6812MINI-E -> Keyboard Switches & Encoders:SK6812MINI-E
- RGB2: renamed from LED5; footprint kicad-keyboard-parts:MX_SK6812MINI-E -> Keyboard Switches & Encoders:RGB_SK6812MINI-E; symbol Keyboard_Library:SK6812MINI-E -> Keyboard Switches & Encoders:SK6812MINI-E
- RGB3: renamed from LED2; footprint kicad-keyboard-parts:MX_SK6812MINI-E -> Keyboard Switches & Encoders:RGB_SK6812MINI-E; symbol Keyboard_Library:SK6812MINI-E -> Keyboard Switches & Encoders:SK6812MINI-E
- RGB4: renamed from LED6; footprint kicad-keyboard-parts:MX_SK6812MINI-E -> Keyboard Switches & Encoders:RGB_SK6812MINI-E; symbol Keyboard_Library:SK6812MINI-E -> Keyboard Switches & Encoders:SK6812MINI-E
- RGB5: renamed from LED3; footprint kicad-keyboard-parts:MX_SK6812MINI-E -> Keyboard Switches & Encoders:RGB_SK6812MINI-E; symbol Keyboard_Library:SK6812MINI-E -> Keyboard Switches & Encoders:SK6812MINI-E
- RGB6: renamed from LED7; footprint kicad-keyboard-parts:MX_SK6812MINI-E -> Keyboard Switches & Encoders:RGB_SK6812MINI-E; symbol Keyboard_Library:SK6812MINI-E -> Keyboard Switches & Encoders:SK6812MINI-E
- RGB7: renamed from LED4; footprint kicad-keyboard-parts:MX_SK6812MINI-E -> Keyboard Switches & Encoders:RGB_SK6812MINI-E; symbol Keyboard_Library:SK6812MINI-E -> Keyboard Switches & Encoders:SK6812MINI-E
- RGB8: renamed from LED8; footprint kicad-keyboard-parts:MX_SK6812MINI-E -> Keyboard Switches & Encoders:RGB_SK6812MINI-E; symbol Keyboard_Library:SK6812MINI-E -> Keyboard Switches & Encoders:SK6812MINI-E
- S1: footprint MSK12C02 -> Keyboard Switches & Encoders:MSK12C02; symbol Keyboard Library:MSK12C02 -> Keyboard Switches & Encoders:MSK12C02
- U1: value ProMicro -> (none); footprint Keebio-Parts:ArduinoProMicro -> (none)
Connections:
- net GND: now also SW1.2, SW2.2, SW3.2, SW4.2, SW5.2, SW6.2
- net Key1: now also U1.8 (C6), SW1.1; no longer U1.7 (D4)
- net Key2: now also U1.10 (E6), SW2.1; no longer U1.9 (D7)
- net Key3: now also U1.12 (B5), SW3.1; no longer U1.11 (B4)
- net Key4: now also U1.7 (D4), SW4.1; no longer U1.8 (C6)
- net Key5: now also U1.9 (D7), SW5.1; no longer U1.10 (E6)
- net Key6: now also U1.11 (B4), SW6.1; no longer U1.12 (B5)
Other:
- moved on the sheet: Logo2
