File: Little Big Scroll 6/Rear Plate/LBS6_Rear_Plate.kicad_pcb (KiCad board)
At the start: 2 copper layers, 57.2 x 85 mm, 6 parts

Commit message: LBS6 v1.01
Parts:
- H1, H2, H3, H4: footprint MountingHole:MountingHole_3.7mm -> MountingHole:MountingHole_2.5mm
Other:
- board text added: "Little Big Scroll 6 - v1.1 Markus Knutsson 2022 https://github.com/TweetyDaBird"
- board text removed: "Little Big Scroll 6 - v1.0 Markus Knutsson 2022 https://github.com/TweetyDaBird"
Changed lines of the file:
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@@
   (title_block
     (title "Little Big Scroll 6")
-    (date "2022-01-28")
-    (rev "v1.0")
+    (date "2022-02-26")
+    (rev "v1.1")
     (company "Tweety's Wild Thinking")
     (comment 1 "Markus Knutsson <markus.knutsson@tweety.se>")
@@
   )
   (net 0 "")
-  (footprint "MountingHole:MountingHole_3.7mm" (layer "F.Cu")
+  (footprint "MountingHole:MountingHole_2.5mm" (layer "F.Cu")
     (at 86.22 112.685)
-    (descr "Mounting Hole 3.7mm, no annular")
-    (tags "mounting hole 3.7mm no annular")
+    (descr "Mounting Hole 2.5mm, no annular")
+    (tags "mounting hole 2.5mm no annular")
     (property "Sheetfile" "LBS6_Rear_Plate.kicad_sch")
     (property "Sheetname" "")
     (attr exclude_from_pos_files)
-    (fp_text reference "H1" (at 0 -4.7) (layer "F.SilkS") hide
+    (fp_text reference "H1" (at 0 -3.5) (layer "F.SilkS")
       (effects (font (size 1 1) (thickness 0.15)))
     )
-    (fp_text value "Hole_PCB_M2-Spacer" (at 0 4.7) (layer "F.Fab")
+    (fp_text value "Hole_PCB_M2-Spacer" (at 0 3.5) (layer "F.Fab")
       (effects (font (size 1 1) (thickness 0.15)))
     )
@@
       (effects (font (size 1 1) (thickness 0.15)))
     )
-    (fp_circle (center 0 0) (end 3.7 0) (layer "Cmts.User") (width 0.15) (fill none))
-    (fp_circle (center 0 0) (end 3.95 0) (layer "F.CrtYd") (width 0.05) (fill none))
-    (pad "" np_thru_hole circle locked (at 0 0) (size 3.7 3.7) (drill 3.7) (layers *.Cu *.Mask))
+    (fp_circle (center 0 0) (end 2.5 0) (layer "Cmts.User") (width 0.15) (fill none))
+    (fp_circle (center 0 0) (end 2.75 0) (layer "F.CrtYd") (width 0.05) (fill none))
+    (pad "" np_thru_hole circle locked (at 0 0) (size 2.5 2.5) (drill 2.5) (layers *.Cu *.Mask))
   )
-  (footprint "MountingHole:MountingHole_3.7mm" (layer "F.Cu")
+  (footprint "MountingHole:MountingHole_2.5mm" (layer "F.Cu")
     (at 134.32 112.685)
-    (descr "Mounting Hole 3.7mm, no annular")
-    (tags "mounting hole 3.7mm no annular")
+    (descr "Mounting Hole 2.5mm, no annular")
+    (tags "mounting hole 2.5mm no annular")
     (property "Sheetfile" "LBS6_Rear_Plate.kicad_sch")
     (property "Sheetname" "")
     (attr exclude_from_pos_files)
-    (fp_text reference "H2" (at 0 -4.7) (layer "F.SilkS") hide
+    (fp_text reference "H2" (at 0 -3.5) (layer "F.SilkS")
       (effects (font (size 1 1) (thickness 0.15)))
     )
-    (fp_text value "Hole_PCB_M2-Spacer" (at 0 4.7) (layer "F.Fab")
+    (fp_text value "Hole_PCB_M2-Spacer" (at 0 3.5) (layer "F.Fab")
       (effects (font (size 1 1) (thickness 0.15)))
     )
@@
       (effects (font (size 1 1) (thickness 0.15)))
     )
-    (fp_circle (center 0 0) (end 3.7 0) (layer "Cmts.User") (width 0.15) (fill none))
-    (fp_circle (center 0 0) (end 3.95 0) (layer "F.CrtYd") (width 0.05) (fill none))
-    (pad "" np_thru_hole circle locked (at 0 0) (size 3.7 3.7) (drill 3.7) (layers *.Cu *.Mask))
+    (fp_circle (center 0 0) (end 2.5 0) (layer "Cmts.User") (width 0.15) (fill none))
+    (fp_circle (center 0 0) (end 2.75 0) (layer "F.CrtYd") (width 0.05) (fill none))
+    (pad "" np_thru_hole circle locked (at 0 0) (size 2.5 2.5) (drill 2.5) (layers *.Cu *.Mask))
   )
-  (footprint "MountingHole:MountingHole_3.7mm" (layer "F.Cu")
+  (footprint "MountingHole:MountingHole_2.5mm" (layer "F.Cu")
     (at 134.94 50.73)
-    (descr "Mounting Hole 3.7mm, no annular")
-    (tags "mounting hole 3.7mm no annular")
+    (descr "Mounting Hole 2.5mm, no annular")
+    (tags "mounting hole 2.5mm no annular")
     (property "Sheetfile" "LBS6_Rear_Plate.kicad_sch")
     (property "Sheetname" "")
     (attr exclude_from_pos_files)
-    (fp_text reference "H3" (at 0 -4.7) (layer "F.SilkS") hide
+    (fp_text reference "H3" (at 0 -3.5) (layer "F.SilkS")
       (effects (font (size 1 1) (thickness 0.15)))
     )
-    (fp_text value "Hole_PCB_M2-Spacer" (at 0 4.7) (layer "F.Fab")
+    (fp_text value "Hole_PCB_M2-Spacer" (at 0 3.5) (layer "F.Fab")
       (effects (font (size 1 1) (thickness 0.15)))
     )
@@
       (effects (font (size 1 1) (thickness 0.15)))
     )
-    (fp_circle (center 0 0) (end 3.7 0) (layer "Cmts.User") (width 0.15) (fill none))
-    (fp_circle (center 0 0) (end 3.95 0) (layer "F.CrtYd") (width 0.05) (fill none))
-    (pad "" np_thru_hole circle locked (at 0 0) (size 3.7 3.7) (drill 3.7) (layers *.Cu *.Mask))
+    (fp_circle (center 0 0) (end 2.5 0) (layer "Cmts.User") (width 0.15) (fill none))
+    (fp_circle (center 0 0) (end 2.75 0) (layer "F.CrtYd") (width 0.05) (fill none))
+    (pad "" np_thru_hole circle locked (at 0 0) (size 2.5 2.5) (drill 2.5) (layers *.Cu *.Mask))
   )
-  (footprint "MountingHole:MountingHole_3.7mm" (layer "F.Cu")
+  (footprint "MountingHole:MountingHole_2.5mm" (layer "F.Cu")
     (at 85.6 50.73)
-    (descr "Mounting Hole 3.7mm, no annular")
-    (tags "mounting hole 3.7mm no annular")
+    (descr "Mounting Hole 2.5mm, no annular")
+    (tags "mounting hole 2.5mm no annular")
     (property "Sheetfile" "LBS6_Rear_Plate.kicad_sch")
     (property "Sheetname" "")
     (attr exclude_from_pos_files)
-    (fp_text reference "H4" (at 0 -4.7) (layer "F.SilkS") hide
+    (fp_text reference "H4" (at 0 -3.5) (layer "F.SilkS")
       (effects (font (size 1 1) (thickness 0.15)))
     )
-    (fp_text value "Hole_PCB_M2-Spacer" (at 0 4.7) (layer "F.Fab")
+    (fp_text value "Hole_PCB_M2-Spacer" (at 0 3.5) (layer "F.Fab")
       (effects (font (size 1 1) (thickness 0.15)))
     )
@@
       (effects (font (size 1 1) (thickness 0.15)))
     )
-    (fp_circle (center 0 0) (end 3.7 0) (layer "Cmts.User") (width 0.15) (fill none))
-    (fp_circle (center 0 0) (end 3.95 0) (layer "F.CrtYd") (width 0.05) (fill none))
-    (pad "" np_thru_hole circle locked (at 0 0) (size 3.7 3.7) (drill 3.7) (layers *.Cu *.Mask))
+    (fp_circle (center 0 0) (end 2.5 0) (layer "Cmts.User") (width 0.15) (fill none))
+    (fp_circle (center 0 0) (end 2.75 0) (layer "F.CrtYd") (width 0.05) (fill none))
+    (pad "" np_thru_hole circle locked (at 0 0) (size 2.5 2.5) (drill 2.5) (layers *.Cu *.Mask))
   )
   (footprint "QMK Logo:Powered_by_QMK" (layer "F.Cu")
@@
     (effects (font (size 0.8 0.8) (thickness 0.15)))
   )
-  (gr_text "Little Big Scroll 6 - v1.0\nMarkus Knutsson 2022\nhttps://github.com/TweetyDaBird" (at 111.16 90.69) (layer "F.SilkS")
+  (gr_text "Little Big Scroll 6 - v1.1\nMarkus Knutsson 2022\nhttps://github.com/TweetyDaBird" (at 111.16 90.69) (layer "F.SilkS")
     (effects (font (size 0.8 0.8) (thickness 0.15)))
   )

Commit message: LSB6 1.01
Parts:
- removed Lic1: CC-BY-SA-4.0, CC_Licensing:CC_BY_SA_40
- removed Logo1: QMK_Logo, QMK Logo:Powered_by_QMK
- H1, H2, H3, H4: value Hole_PCB_M2-Spacer -> Spacer_Plate
- moved H1 1.62 mm to (84.6, 112.7)
- moved H2 1.62 mm to (135.9, 112.7)
- moved H3 1.41 mm to (135.9, 49.7)
- moved H4 1.41 mm to (84.6, 49.7)
Routing:
- added copper zone on B.Cu, net (none)
- added copper zone on F.Cu, net (none)
Other:
- board size 57.2 x 85 mm -> 59.2 x 87 mm
- board text removed: "JLCJLCJLCJLC"
- board text removed: "Little Big Scroll 6 - v1.1 Markus Knutsson 2022 https://github.com/TweetyDaBird"
