File: Little Big Scroll 6/Rear Plate/LBS6_Rear_Plate.kicad_sch (KiCad schematic)
At the start: 6 parts

Commit message: LBS6 v1.01
Parts:
- H1, H2, H3, H4: footprint MountingHole:MountingHole_3.7mm -> MountingHole:MountingHole_2.5mm
Changed lines of the file:
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@@
       (effects (font (size 1.524 1.524)) (justify left))
     )
-    (property "Footprint" "MountingHole:MountingHole_3.7mm" (id 2) (at 29.21 189.23 0)
+    (property "Footprint" "MountingHole:MountingHole_2.5mm" (id 2) (at 29.21 189.23 0)
       (effects (font (size 1.524 1.524)) hide)
     )
@@
       (effects (font (size 1.524 1.524)) (justify left))
     )
-    (property "Footprint" "MountingHole:MountingHole_3.7mm" (id 2) (at 29.21 168.91 0)
+    (property "Footprint" "MountingHole:MountingHole_2.5mm" (id 2) (at 29.21 168.91 0)
       (effects (font (size 1.524 1.524)) hide)
     )
@@
       (effects (font (size 1.524 1.524)) (justify left))
     )
-    (property "Footprint" "MountingHole:MountingHole_3.7mm" (id 2) (at 29.21 158.75 0)
+    (property "Footprint" "MountingHole:MountingHole_2.5mm" (id 2) (at 29.21 158.75 0)
       (effects (font (size 1.524 1.524)) hide)
     )
@@
       (effects (font (size 1.524 1.524)) (justify left))
     )
-    (property "Footprint" "MountingHole:MountingHole_3.7mm" (id 2) (at 29.21 179.07 0)
+    (property "Footprint" "MountingHole:MountingHole_2.5mm" (id 2) (at 29.21 179.07 0)
       (effects (font (size 1.524 1.524)) hide)
     )
@@
   (symbol_instances
     (path "/00000000-0000-0000-0000-000061f277e9"
-      (reference "H1") (unit 1) (value "Hole_PCB_M2-Spacer") (footprint "MountingHole:MountingHole_3.7mm")
+      (reference "H1") (unit 1) (value "Hole_PCB_M2-Spacer") (footprint "MountingHole:MountingHole_2.5mm")
     )
     (path "/00000000-0000-0000-0000-000061f26e99"
-      (reference "H2") (unit 1) (value "Hole_PCB_M2-Spacer") (footprint "MountingHole:MountingHole_3.7mm")
+      (reference "H2") (unit 1) (value "Hole_PCB_M2-Spacer") (footprint "MountingHole:MountingHole_2.5mm")
     )
     (path "/00000000-0000-0000-0000-000061f28116"
-      (reference "H3") (unit 1) (value "Hole_PCB_M2-Spacer") (footprint "MountingHole:MountingHole_3.7mm")
+      (reference "H3") (unit 1) (value "Hole_PCB_M2-Spacer") (footprint "MountingHole:MountingHole_2.5mm")
     )
     (path "/00000000-0000-0000-0000-000061f26001"
-      (reference "H4") (unit 1) (value "Hole_PCB_M2-Spacer") (footprint "MountingHole:MountingHole_3.7mm")
+      (reference "H4") (unit 1) (value "Hole_PCB_M2-Spacer") (footprint "MountingHole:MountingHole_2.5mm")
     )
     (path "/0cbbf3d2-db89-46d7-9721-0bda6fb9d450"

Commit message: LSB6 1.01
Parts:
- H1, H2, H3, H4: value Hole_PCB_M2-Spacer -> Spacer_Plate; symbol Keyboard_Library:Hole_PCB_M2-Spacer -> Keyboard Switches & Encoders:Spacer_Plate
- Logo1: renamed from Lic1; footprint CC_Licensing:CC_BY_SA_40 -> Logotypes:CC_BY_SA_40; symbol CC_Licensing:CC-BY-SA-4.0 -> Logotypes:CC-BY-SA-4.0
- Logo2: renamed from Logo1; footprint QMK Logo:Powered_by_QMK -> Logotypes:Powered_by_QMK; symbol Keyboard Library:QMK_Logo -> Logotypes:QMK_Logo; now left out of the parts list
Other:
- moved on the sheet: Logo2
Changed lines of the file:
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@@
   (title_block
     (title "Little Big Scroll 6")
-    (date "2022-01-28")
-    (rev "v1.0")
+    (date "2022-04-07")
+    (rev "v1.01")
     (company "Tweety's Wild Thinking")
     (comment 1 "Markus Knutsson <markus.knutsson@tweety.se>")
@@
     (comment 3 "Licensed under Creative Commons BY-SA 4.0 International")
   )
-  (symbol (lib_id "Keyboard_Library:Hole_PCB_M2-Spacer") (at 29.21 189.23 0) (unit 1)
+  (symbol (lib_id "Keyboard Switches & Encoders:Spacer_Plate") (at 29.21 189.23 0) (unit 1)
     (in_bom yes) (on_board yes)
     (property "Reference" "H4" (id 0) (at 33.9344 187.8838 0)
       (effects (font (size 1.524 1.524)) (justify left))
     )
-    (property "Value" "Hole_PCB_M2-Spacer" (id 1) (at 33.9344 190.5762 0)
+    (property "Value" "Spacer_Plate" (id 1) (at 33.9344 190.5762 0)
       (effects (font (size 1.524 1.524)) (justify left))
     )
@@
     )
   )
-  (symbol (lib_id "Keyboard_Library:Hole_PCB_M2-Spacer") (at 29.21 168.91 0) (unit 1)
+  (symbol (lib_id "Keyboard Switches & Encoders:Spacer_Plate") (at 29.21 168.91 0) (unit 1)
     (in_bom yes) (on_board yes)
     (property "Reference" "H2" (id 0) (at 33.9344 167.5638 0)
       (effects (font (size 1.524 1.524)) (justify left))
     )
-    (property "Value" "Hole_PCB_M2-Spacer" (id 1) (at 33.9344 170.2562 0)
+    (property "Value" "Spacer_Plate" (id 1) (at 33.9344 170.2562 0)
       (effects (font (size 1.524 1.524)) (justify left))
     )
@@
     )
   )
-  (symbol (lib_id "Keyboard_Library:Hole_PCB_M2-Spacer") (at 29.21 158.75 0) (unit 1)
+  (symbol (lib_id "Keyboard Switches & Encoders:Spacer_Plate") (at 29.21 158.75 0) (unit 1)
     (in_bom yes) (on_board yes)
     (property "Reference" "H1" (id 0) (at 33.9344 157.4038 0)
       (effects (font (size 1.524 1.524)) (justify left))
     )
-    (property "Value" "Hole_PCB_M2-Spacer" (id 1) (at 33.9344 160.0962 0)
+    (property "Value" "Spacer_Plate" (id 1) (at 33.9344 160.0962 0)
       (effects (font (size 1.524 1.524)) (justify left))
     )
@@
     )
   )
-  (symbol (lib_id "Keyboard_Library:Hole_PCB_M2-Spacer") (at 29.21 179.07 0) (unit 1)
+  (symbol (lib_id "Keyboard Switches & Encoders:Spacer_Plate") (at 29.21 179.07 0) (unit 1)
     (in_bom yes) (on_board yes)
     (property "Reference" "H3" (id 0) (at 33.9344 177.7238 0)
       (effects (font (size 1.524 1.524)) (justify left))
     )
-    (property "Value" "Hole_PCB_M2-Spacer" (id 1) (at 33.9344 180.4162 0)
+    (property "Value" "Spacer_Plate" (id 1) (at 33.9344 180.4162 0)
       (effects (font (size 1.524 1.524)) (justify left))
     )
@@
     )
   )
-  (symbol (lib_id "CC_Licensing:CC-BY-SA-4.0") (at 97.79 177.8 0) (unit 1)
+  (symbol (lib_id "Logotypes:CC-BY-SA-4.0") (at 97.79 177.8 0) (unit 1)
     (in_bom yes) (on_board yes) (fields_autoplaced)
-    (property "Reference" "Lic1" (id 0) (at 97.79 171.4205 0))
-    (property "Value" "CC-BY-SA-4.0" (id 1) (at 97.79 174.1956 0))
-    (property "Footprint" "CC_Licensing:CC_BY_SA_40" (id 2) (at 97.79 177.8 0)
+    (property "Reference" "Logo1" (id 0) (at 97.79 176.53 0))
+    (property "Value" "CC-BY-SA-4.0" (id 1) (at 97.79 179.07 0))
+    (property "Footprint" "Logotypes:CC_BY_SA_40" (id 2) (at 97.79 177.8 0)
       (effects (font (size 1.27 1.27)) hide)
     )
@@
     )
   )
-  (symbol (lib_id "Keyboard Library:QMK_Logo") (at 128.27 179.07 0) (unit 1)
-    (in_bom yes) (on_board yes) (fields_autoplaced)
-    (property "Reference" "Logo1" (id 0) (at 132.9182 178.0053 0)
-      (effects (font (size 1.524 1.524)) (justify left))
-    )
-    (property "Value" "QMK_Logo" (id 1) (at 132.9182 181.2843 0)
-      (effects (font (size 1.524 1.524)) (justify left))
-    )
-    (property "Footprint" "QMK Logo:Powered_by_QMK" (id 2) (at 128.27 179.07 0)
-      (effects (font (size 1.524 1.524)) hide)
+  (symbol (lib_id "Logotypes:QMK_Logo") (at 128.27 179.07 0) (unit 1)
+    (in_bom no) (on_board yes) (fields_autoplaced)
+    (property "Reference" "Logo2" (id 0) (at 128.27 179.07 0))
+    (property "Value" "QMK_Logo" (id 1) (at 128.27 176.53 0))
+    (property "Footprint" "Logotypes:Powered_by_QMK" (id 2) (at 128.27 179.07 0)
+      (effects (font (size 1.27 1.27)) hide)
     )
     (property "Datasheet" "" (id 3) (at 128.27 179.07 0)
-      (effects (font (size 1.524 1.524)) hide)
+      (effects (font (size 1.27 1.27)) hide)
     )
   )
@@
   (symbol_instances
     (path "/00000000-0000-0000-0000-000061f277e9"
-      (reference "H1") (unit 1) (value "Hole_PCB_M2-Spacer") (footprint "MountingHole:MountingHole_2.5mm")
+      (reference "H1") (unit 1) (value "Spacer_Plate") (footprint "MountingHole:MountingHole_2.5mm")
     )
     (path "/00000000-0000-0000-0000-000061f26e99"
-      (reference "H2") (unit 1) (value "Hole_PCB_M2-Spacer") (footprint "MountingHole:MountingHole_2.5mm")
+      (reference "H2") (unit 1) (value "Spacer_Plate") (footprint "MountingHole:MountingHole_2.5mm")
     )
     (path "/00000000-0000-0000-0000-000061f28116"
-      (reference "H3") (unit 1) (value "Hole_PCB_M2-Spacer") (footprint "MountingHole:MountingHole_2.5mm")
+      (reference "H3") (unit 1) (value "Spacer_Plate") (footprint "MountingHole:MountingHole_2.5mm")
     )
     (path "/00000000-0000-0000-0000-000061f26001"
-      (reference "H4") (unit 1) (value "Hole_PCB_M2-Spacer") (footprint "MountingHole:MountingHole_2.5mm")
+      (reference "H4") (unit 1) (value "Spacer_Plate") (footprint "MountingHole:MountingHole_2.5mm")
     )
     (path "/0cbbf3d2-db89-46d7-9721-0bda6fb9d450"
-      (reference "Lic1") (unit 1) (value "CC-BY-SA-4.0") (footprint "CC_Licensing:CC_BY_SA_40")
+      (reference "Logo1") (unit 1) (value "CC-BY-SA-4.0") (footprint "Logotypes:CC_BY_SA_40")
     )
     (path "/12afcaef-113a-42be-8bf9-dd3ec0296311"
-      (reference "Logo1") (unit 1) (value "QMK_Logo") (footprint "QMK Logo:Powered_by_QMK")
+      (reference "Logo2") (unit 1) (value "QMK_Logo") (footprint "Logotypes:Powered_by_QMK")
     )
   )
