File: Little Big Scroll 6/prototype/PCB/Little Big Scroll 6 - PCB.kicad_pcb (KiCad board)
At the start: 2 copper layers, 59.2 x 87 mm, 27 parts, among them J1 Conn_01x02, J2 Conn_01x02, SW1 SW_MX_HS, SW2 SW_MX_HS, SW3 SW_MX_HS, SW4 SW_MX_HS, SW5 SW_MX_HS, SW6 SW_MX_HS, U1 ProMicro

Commit message: LSB6 Prototype v1.1
Parts:
- moved C1 1.76 mm to (107.8, 71.6)
- moved C2 1.72 mm to (112.8, 64.1)
Routing:
- net EncKey: track 16.3 -> 21.1 mm
- net VCC: track 197.5 -> 194.8 mm
- net EncB: track 13.8 -> 15.8 mm
- net EncA: track 7.70 -> 9.53 mm
Other:
- board text added: "1. Solder hotswap sockets from rear of PCB, follow outline 2. Solder capacitors (C1 & C2) from rear (unidirectional) 3. Cut ends of legs flush on front side (underneath encoder) 4. Solder RGB from rear, orient by arrow/marked leg 5. Solder controller on rear of PCB, facing up 6. Solder encoder from front of PCB (Bend ground tabs!) 7. Assemble, Flash and Enjoy!"
- board text added: "Little Big Scroll 6 - v1.1 Markus Knutsson 2022 https://github.com/TweetyDaBird"
- board text removed: "1. Solder hotswap sockets from rear of PCB, follow outline 2. Solder capacitors (C1 & C2) from rear (unidirectional) 3. Cut ends of legs flush on front side underneath encoder 4. Solder RGB from rear, orient by arrow/cut leg corner 5. Solder controller from rear, facing up 6. Solder encoder from front of PCB 7. Assemble, Flash and Enjoy!"
- board text removed: "Little Big Scroll 6 - v1.02 Markus Knutsson 2022 https://github.com/TweetyDaBird"
