File: Little Big Scroll 6/v1.1.1/Front Plate/Little Big Scroll 6 - Front Plate.kicad_sch (KiCad schematic)
At the start: 15 parts, among them SW1 SW_MX_HS, SW2 SW_MX_HS, SW3 SW_MX_HS, SW4 SW_MX_HS, SW5 SW_MX_HS, SW6 SW_MX_HS

Commit message: LBS6 v1.1.1
Fixed plate holes
Parts:
- H1, H2, H3, H4: footprint Keyboard Switches & Encoders:Spacer PCB hole -> Keyboard_Plate:Spacer Plate hole; symbol Keyboard Switches & Encoders:Spacer_PCB -> Keyboard_Plate:Spacer_Plate
Changed lines of the file:
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@@
     (pin "4")
   )
-  (symbol (lib_id "Keyboard Switches & Encoders:Spacer_PCB") (at 29.21 189.23 0) (unit 1)
+  (symbol (lib_id "Keyboard_Plate:Spacer_Plate") (at 29.21 189.23 0) (unit 1)
     (in_bom yes) (on_board yes)
     (property "Reference" "H4" (id 0) (at 29.21 190.5 0)
@@
       (effects (font (size 1.524 1.524)))
     )
-    (property "Footprint" "Keyboard Switches & Encoders:Spacer PCB hole" (id 2) (at 29.21 189.23 0)
+    (property "Footprint" "Keyboard_Plate:Spacer Plate hole" (id 2) (at 29.21 189.23 0)
       (effects (font (size 1.524 1.524)) hide)
     )
@@
     )
   )
-  (symbol (lib_id "Keyboard Switches & Encoders:Spacer_PCB") (at 29.21 168.91 0) (unit 1)
+  (symbol (lib_id "Keyboard_Plate:Spacer_Plate") (at 29.21 168.91 0) (unit 1)
     (in_bom yes) (on_board yes)
     (property "Reference" "H2" (id 0) (at 29.21 170.18 0)
@@
       (effects (font (size 1.524 1.524)))
     )
-    (property "Footprint" "Keyboard Switches & Encoders:Spacer PCB hole" (id 2) (at 29.21 168.91 0)
+    (property "Footprint" "Keyboard_Plate:Spacer Plate hole" (id 2) (at 29.21 168.91 0)
       (effects (font (size 1.524 1.524)) hide)
     )
@@
     )
   )
-  (symbol (lib_id "Keyboard Switches & Encoders:Spacer_PCB") (at 29.21 158.75 0) (unit 1)
+  (symbol (lib_id "Keyboard_Plate:Spacer_Plate") (at 29.21 158.75 0) (unit 1)
     (in_bom yes) (on_board yes)
     (property "Reference" "H1" (id 0) (at 29.21 160.02 0)
@@
       (effects (font (size 1.524 1.524)))
     )
-    (property "Footprint" "Keyboard Switches & Encoders:Spacer PCB hole" (id 2) (at 29.21 158.75 0)
+    (property "Footprint" "Keyboard_Plate:Spacer Plate hole" (id 2) (at 29.21 158.75 0)
       (effects (font (size 1.524 1.524)) hide)
     )
@@
     )
   )
-  (symbol (lib_id "Keyboard Switches & Encoders:Spacer_PCB") (at 29.21 179.07 0) (unit 1)
+  (symbol (lib_id "Keyboard_Plate:Spacer_Plate") (at 29.21 179.07 0) (unit 1)
     (in_bom yes) (on_board yes)
     (property "Reference" "H3" (id 0) (at 29.21 180.34 0)
@@
       (effects (font (size 1.524 1.524)))
     )
-    (property "Footprint" "Keyboard Switches & Encoders:Spacer PCB hole" (id 2) (at 29.21 179.07 0)
+    (property "Footprint" "Keyboard_Plate:Spacer Plate hole" (id 2) (at 29.21 179.07 0)
       (effects (font (size 1.524 1.524)) hide)
     )
@@
     )
     (path "/00000000-0000-0000-0000-000061f277e9"
-      (reference "H1") (unit 1) (value "Spacer_PCB") (footprint "Keyboard Switches & Encoders:Spacer PCB hole")
+      (reference "H1") (unit 1) (value "Spacer_PCB") (footprint "Keyboard_Plate:Spacer Plate hole")
     )
     (path "/00000000-0000-0000-0000-000061f26e99"
-      (reference "H2") (unit 1) (value "Spacer_PCB") (footprint "Keyboard Switches & Encoders:Spacer PCB hole")
+      (reference "H2") (unit 1) (value "Spacer_PCB") (footprint "Keyboard_Plate:Spacer Plate hole")
     )
     (path "/00000000-0000-0000-0000-000061f28116"
-      (reference "H3") (unit 1) (value "Spacer_PCB") (footprint "Keyboard Switches & Encoders:Spacer PCB hole")
+      (reference "H3") (unit 1) (value "Spacer_PCB") (footprint "Keyboard_Plate:Spacer Plate hole")
     )
     (path "/00000000-0000-0000-0000-000061f26001"
-      (reference "H4") (unit 1) (value "Spacer_PCB") (footprint "Keyboard Switches & Encoders:Spacer PCB hole")
+      (reference "H4") (unit 1) (value "Spacer_PCB") (footprint "Keyboard_Plate:Spacer Plate hole")
     )
     (path "/0cbbf3d2-db89-46d7-9721-0bda6fb9d450"
