File: Little Big Scroll 6/v1.1.1/PCB/Little Big Scroll 6 - PCB.kicad_pcb (KiCad board)
At the start: 2 copper layers, 59.2 x 87 mm, 27 parts, among them J1 Conn_01x02, J2 Conn_01x02, SW1 SW_MX_HS, SW2 SW_MX_HS, SW3 SW_MX_HS, SW4 SW_MX_HS, SW5 SW_MX_HS, SW6 SW_MX_HS, U1 ProMicro

Commit message: LBS6 v1.1.1
Fixed plate holes
Parts:
- ENC1: footprint Keyboard Switches & Encoders:Encoder_Alps_EC11E_Small -> Keyboard Encoders:Encoder_Alps_EC11E_Small
- H1, H2, H3, H4: footprint Keyboard Switches & Encoders:Spacer PCB hole -> Keyboard Common:Spacer PCB hole
- S1: footprint Keyboard Switches & Encoders:MSK12C02 -> Keyboard Common:MSK12C02
Other:
- board text added: "Little Big Scroll 6 - v1.1.1 Markus Knutsson 2022 https://github.com/TweetyDaBird"
- board text removed: "Little Big Scroll 6 - v1.1 Markus Knutsson 2022 https://github.com/TweetyDaBird"
