File: Little Big Scroll 6/v1.1.1/PCB/Little Big Scroll 6 - PCB.kicad_sch (KiCad schematic)
At the start: 27 parts, among them J1 Conn_01x02, J2 Conn_01x02, SW1 SW_MX_HS, SW2 SW_MX_HS, SW3 SW_MX_HS, SW4 SW_MX_HS, SW5 SW_MX_HS, SW6 SW_MX_HS, U1 ProMicro

Commit message: LBS6 v1.1.1
Fixed plate holes
Parts:
- ENC1: footprint Keyboard Switches & Encoders:Encoder_Alps_EC11E_Small -> Keyboard Encoders:Encoder_Alps_EC11E_Small; symbol Keyboard Switches & Encoders:Rotary_Encoder_Click -> Keyboard Switches:Rotary_Encoder_Click
- H1, H2, H3, H4: symbol Keyboard Switches & Encoders:Spacer_PCB -> Keyboard_Plate:Spacer_PCB
- RGB1, RGB2, RGB3, RGB4, RGB5, RGB6, RGB7, RGB8: symbol Keyboard Switches & Encoders:SK6812MINI-E -> Keyboard Common:SK6812MINI-E
- S1: footprint Keyboard Switches & Encoders:MSK12C02 -> Keyboard Common:MSK12C02; symbol Keyboard Switches & Encoders:MSK12C02 -> Keyboard Common:MSK12C02
- SW1, SW2, SW3, SW4, SW5, SW6: symbol Keyboard Switches & Encoders:SW_MX_HS -> Keyboard Switches:SW_MX_HotSwap
- U1: symbol Common Library:ProMicro -> Keyboard Controllers:ProMicro
Changed lines of the file:
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@@
   (title_block
     (title "Little Big Scroll 6 - PCB")
-    (date "2022-08-26")
-    (rev "v1.1")
+    (date "2022-09-16")
+    (rev "v1.1.1")
     (company "Tweety's Wild Thinking")
     (comment 1 "Markus Knutsson <markus.knutsson@tweety.se>")
@@
     )
   )
-  (symbol (lib_id "Common Library:ProMicro") (at 57.15 48.26 0) (unit 1)
+  (symbol (lib_id "Keyboard Controllers:ProMicro") (at 57.15 48.26 0) (unit 1)
     (in_bom yes) (on_board yes)
     (property "Reference" "U1" (id 0) (at 57.15 27.0002 0)
@@
     (pin "9")
   )
-  (symbol (lib_id "Keyboard Switches & Encoders:Rotary_Encoder_Click") (at 60.96 102.87 0) (unit 1)
+  (symbol (lib_id "Keyboard Switches:Rotary_Encoder_Click") (at 60.96 102.87 0) (unit 1)
     (in_bom yes) (on_board yes)
     (property "Reference" "ENC1" (id 0) (at 60.96 96.266 0))
     (property "Value" "Rotary_Encoder_Click" (id 1) (at 60.96 93.98 0))
-    (property "Footprint" "Keyboard Switches & Encoders:Encoder_Alps_EC11E_Small" (id 2) (at 57.15 98.806 0)
+    (property "Footprint" "Keyboard Encoders:Encoder_Alps_EC11E_Small" (id 2) (at 57.15 98.806 0)
       (effects (font (size 1.27 1.27)) hide)
     )
@@
     (pin "1")
   )
-  (symbol (lib_id "Keyboard Switches & Encoders:SK6812MINI-E") (at 179.07 36.83 0) (unit 1)
+  (symbol (lib_id "Keyboard Common:SK6812MINI-E") (at 179.07 36.83 0) (unit 1)
     (in_bom yes) (on_board yes)
     (property "Reference" "RGB1" (id 0) (at 184.15 31.115 0)
@@
     (pin "4")
   )
-  (symbol (lib_id "Keyboard Switches & Encoders:SK6812MINI-E") (at 196.85 36.83 0) (unit 1)
+  (symbol (lib_id "Keyboard Common:SK6812MINI-E") (at 196.85 36.83 0) (unit 1)
     (in_bom yes) (on_board yes)
     (property "Reference" "RGB2" (id 0) (at 201.93 31.115 0)
@@
     (pin "4")
   )
-  (symbol (lib_id "Keyboard Switches & Encoders:SK6812MINI-E") (at 214.63 36.83 0) (unit 1)
+  (symbol (lib_id "Keyboard Common:SK6812MINI-E") (at 214.63 36.83 0) (unit 1)
     (in_bom yes) (on_board yes)
     (property "Reference" "RGB3" (id 0) (at 219.71 31.115 0)
@@
     (pin "4")
   )
-  (symbol (lib_id "Keyboard Switches & Encoders:SK6812MINI-E") (at 179.07 57.15 0) (unit 1)
+  (symbol (lib_id "Keyboard Common:SK6812MINI-E") (at 179.07 57.15 0) (unit 1)
     (in_bom yes) (on_board yes)
     (property "Reference" "RGB5" (id 0) (at 184.15 51.435 0)
@@
     (pin "4")
   )
-  (symbol (lib_id "Keyboard Switches & Encoders:SK6812MINI-E") (at 196.85 57.15 0) (unit 1)
+  (symbol (lib_id "Keyboard Common:SK6812MINI-E") (at 196.85 57.15 0) (unit 1)
     (in_bom yes) (on_board yes)
     (property "Reference" "RGB6" (id 0) (at 201.93 51.435 0)
@@
     (pin "4")
   )
-  (symbol (lib_id "Keyboard Switches & Encoders:SK6812MINI-E") (at 214.63 57.15 0) (unit 1)
+  (symbol (lib_id "Keyboard Common:SK6812MINI-E") (at 214.63 57.15 0) (unit 1)
     (in_bom yes) (on_board yes)
     (property "Reference" "RGB7" (id 0) (at 219.71 51.435 0)
@@
     (pin "4")
   )
-  (symbol (lib_id "Keyboard Switches & Encoders:SK6812MINI-E") (at 232.41 36.83 0) (unit 1)
+  (symbol (lib_id "Keyboard Common:SK6812MINI-E") (at 232.41 36.83 0) (unit 1)
     (in_bom yes) (on_board yes)
     (property "Reference" "RGB4" (id 0) (at 237.49 31.115 0)
@@
     (pin "4")
   )
-  (symbol (lib_id "Keyboard Switches & Encoders:SK6812MINI-E") (at 232.41 57.15 0) (unit 1)
+  (symbol (lib_id "Keyboard Common:SK6812MINI-E") (at 232.41 57.15 0) (unit 1)
     (in_bom yes) (on_board yes)
     (property "Reference" "RGB8" (id 0) (at 237.49 51.435 0)
@@
     (pin "1")
   )
-  (symbol (lib_id "Keyboard Switches & Encoders:Spacer_PCB") (at 29.21 189.23 0) (unit 1)
+  (symbol (lib_id "Keyboard_Plate:Spacer_PCB") (at 29.21 189.23 0) (unit 1)
     (in_bom yes) (on_board yes)
     (property "Reference" "H4" (id 0) (at 29.21 190.5 0)
@@
     )
   )
-  (symbol (lib_id "Keyboard Switches & Encoders:Spacer_PCB") (at 29.21 168.91 0) (unit 1)
+  (symbol (lib_id "Keyboard_Plate:Spacer_PCB") (at 29.21 168.91 0) (unit 1)
     (in_bom yes) (on_board yes)
     (property "Reference" "H2" (id 0) (at 29.21 170.18 0)
@@
     )
   )
-  (symbol (lib_id "Keyboard Switches & Encoders:Spacer_PCB") (at 29.21 158.75 0) (unit 1)
+  (symbol (lib_id "Keyboard_Plate:Spacer_PCB") (at 29.21 158.75 0) (unit 1)
     (in_bom yes) (on_board yes)
     (property "Reference" "H1" (id 0) (at 29.21 160.02 0)
@@
     )
   )
-  (symbol (lib_id "Keyboard Switches & Encoders:Spacer_PCB") (at 29.21 179.07 0) (unit 1)
+  (symbol (lib_id "Keyboard_Plate:Spacer_PCB") (at 29.21 179.07 0) (unit 1)
     (in_bom yes) (on_board yes)
     (property "Reference" "H3" (id 0) (at 29.21 180.34 0)
@@
     )
   )
-  (symbol (lib_id "Keyboard Switches & Encoders:SW_MX_HS") (at 125.73 93.98 0) (unit 1)
+  (symbol (lib_id "Keyboard Switches:SW_MX_HotSwap") (at 125.73 93.98 0) (unit 1)
     (in_bom yes) (on_board yes) (fields_autoplaced)
     (property "Reference" "SW1" (id 0) (at 124.46 88.9 0)
@@
     (pin "2")
   )
-  (symbol (lib_id "Keyboard Switches & Encoders:SW_MX_HS") (at 125.73 114.3 0) (unit 1)
+  (symbol (lib_id "Keyboard Switches:SW_MX_HotSwap") (at 125.73 114.3 0) (unit 1)
     (in_bom yes) (on_board yes) (fields_autoplaced)
     (property "Reference" "SW3" (id 0) (at 124.46 109.22 0)
@@
     (pin "1")
   )
-  (symbol (lib_id "Keyboard Switches & Encoders:SW_MX_HS") (at 147.32 93.98 0) (unit 1)
+  (symbol (lib_id "Keyboard Switches:SW_MX_HotSwap") (at 147.32 93.98 0) (unit 1)
     (in_bom yes) (on_board yes) (fields_autoplaced)
     (property "Reference" "SW4" (id 0) (at 146.05 88.9 0)
@@
     (pin "2")
   )
-  (symbol (lib_id "Keyboard Switches & Encoders:SW_MX_HS") (at 125.73 104.14 0) (unit 1)
+  (symbol (lib_id "Keyboard Switches:SW_MX_HotSwap") (at 125.73 104.14 0) (unit 1)
     (in_bom yes) (on_board yes) (fields_autoplaced)
     (property "Reference" "SW2" (id 0) (at 124.46 99.06 0)
@@
     (pin "2")
   )
-  (symbol (lib_id "Keyboard Switches & Encoders:MSK12C02") (at 189.23 107.95 0) (unit 1)
+  (symbol (lib_id "Keyboard Common:MSK12C02") (at 189.23 107.95 0) (unit 1)
     (in_bom yes) (on_board yes) (fields_autoplaced)
     (property "Reference" "S1" (id 0) (at 182.88 100.33 0)
@@
       (effects (font (size 1.27 1.27)) (justify left))
     )
-    (property "Footprint" "Keyboard Switches & Encoders:MSK12C02" (id 2) (at 199.39 101.6 0)
+    (property "Footprint" "Keyboard Common:MSK12C02" (id 2) (at 199.39 101.6 0)
       (effects (font (size 1.27 1.27)) (justify left) hide)
     )
@@
     (pin "2")
   )
-  (symbol (lib_id "Keyboard Switches & Encoders:SW_MX_HS") (at 147.32 104.14 0) (unit 1)
+  (symbol (lib_id "Keyboard Switches:SW_MX_HotSwap") (at 147.32 104.14 0) (unit 1)
     (in_bom yes) (on_board yes) (fields_autoplaced)
     (property "Reference" "SW5" (id 0) (at 146.05 99.06 0)
@@
     (pin "2")
   )
-  (symbol (lib_id "Keyboard Switches & Encoders:SW_MX_HS") (at 147.32 114.3 0) (unit 1)
+  (symbol (lib_id "Keyboard Switches:SW_MX_HotSwap") (at 147.32 114.3 0) (unit 1)
     (in_bom yes) (on_board yes) (fields_autoplaced)
     (property "Reference" "SW6" (id 0) (at 146.05 109.22 0)
@@
     )
     (path "/00000000-0000-0000-0000-000061eb9f5d"
-      (reference "ENC1") (unit 1) (value "Rotary_Encoder_Click") (footprint "Keyboard Switches & Encoders:Encoder_Alps_EC11E_Small")
+      (reference "ENC1") (unit 1) (value "Rotary_Encoder_Click") (footprint "Keyboard Encoders:Encoder_Alps_EC11E_Small")
     )
     (path "/00000000-0000-0000-0000-000061f277e9"
@@
     )
     (path "/7fc6eda3-a41a-4ab9-935d-37e18cb30594"
-      (reference "S1") (unit 1) (value "MSK12C02") (footprint "Keyboard Switches & Encoders:MSK12C02")
+      (reference "S1") (unit 1) (value "MSK12C02") (footprint "Keyboard Common:MSK12C02")
     )
     (path "/0f07bf18-dcb5-4b28-8cb4-1360a13c3013"
