File: Little Big Scroll 4/v2.00/PCB/Little_Big_Scroll_4.kicad_pcb (KiCad board)
At the start: 2 copper layers, 88.6 x 45 mm, 22 parts, among them SW1 SW_Push, SW2 SW_Push, SW3 SW_Push, SW4 SW_Push

Commit message: LSB 4 v2
Initial design
Parts:
- Logo1: footprint Logotypes:CC_BY_SA_40 -> Logotypes:CC_BY_SA_40_line
- RZ1: footprint Keyboard Controllers:RP2040-Zero_reverse_mount -> Keyboard Controllers:RP2040-Zero_castellated
- SW1, SW2, SW3, SW4: footprint keyswitches:Kailh_socket_MX_RGB -> Keyboard Switches:SW_MX_HotSwap
Connections:
- RZ1 pad 22: VCC -> GND
- RZ1 pad 23: GND -> VCC
- SW1 pad 1: GND -> Key1
- SW1 pad 2: Key1 -> GND
- SW2 pad 1: GND -> Key2
- SW2 pad 2: Key2 -> GND
- SW3 pad 1: GND -> Key3
- SW3 pad 2: Key3 -> GND
- SW4 pad 1: GND -> Key4
- SW4 pad 2: Key4 -> GND
Routing:
- net Key4: track 20.5 -> 19.9 mm
- net Key3: track 40.6 -> 40.0 mm
Other:
- outline, holes or cut-outs redrawn
