File: Little Big Scroll 4/v2.00/PCB/Little_Big_Scroll_4.kicad_sch (KiCad schematic)
At the start: 22 parts, among them SW1 SW_Push, SW2 SW_Push, SW3 SW_Push, SW4 SW_Push

Commit message: LSB 4 v2
Initial design
Parts:
- RZ1: footprint Keyboard Controllers:RP2040-Zero_reverse_mount -> Keyboard Controllers:RP2040-Zero
- SW1, SW2, SW3, SW4: footprint (none) -> Keyboard Switches:SW_MX_HotSwap; symbol Switch:SW_Push -> Keyboard Switches:SW_MX_HotSwap
Connections:
- net GND: now also RZ1.22 (GND), SW1.2, SW2.2, SW3.2, SW4.2; no longer RZ1.23 (GND), SW1.1, SW2.1, SW3.1, SW4.1
- net Key1: now also SW1.1; no longer SW1.2
- net Key2: now also SW2.1; no longer SW2.2
- net Key3: now also SW3.1; no longer SW3.2
- net Key4: now also SW4.1; no longer SW4.2
- net VCC: now also RZ1.23 (5V); no longer RZ1.22 (5V)
Changed lines of the file:
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@@
 			)
 		)
-		(property "Footprint" "Keyboard Controllers:RP2040-Zero_reverse_mount"
+		(property "Footprint" "Keyboard Controllers:RP2040-Zero"
 			(at 64.516 55.88 0)
 			(effects
@@
 	)
 	(symbol
-		(lib_id "Switch:SW_Push")
+		(lib_id "Keyboard Switches:SW_MX_HotSwap")
 		(at 148.59 45.72 0)
-		(mirror y)
 		(unit 1)
 		(exclude_from_sim no)
@@
 		(dnp no)
 		(property "Reference" "SW1"
-			(at 147.32 43.18 0)
+			(at 149.86 43.18 0)
 			(effects
 				(font
@@
 			)
 		)
-		(property "Footprint" ""
+		(property "Footprint" "Keyboard Switches:SW_MX_HotSwap"
 			(at 148.59 40.64 0)
 			(effects
@@
 	)
 	(symbol
-		(lib_id "Switch:SW_Push")
+		(lib_id "Keyboard Switches:SW_MX_HotSwap")
 		(at 148.59 55.88 0)
-		(mirror y)
 		(unit 1)
 		(exclude_from_sim no)
@@
 		(dnp no)
 		(property "Reference" "SW2"
-			(at 147.32 53.34 0)
+			(at 149.86 53.34 0)
 			(effects
 				(font
@@
 			)
 		)
-		(property "Footprint" ""
+		(property "Footprint" "Keyboard Switches:SW_MX_HotSwap"
 			(at 148.59 50.8 0)
 			(effects
@@
 	)
 	(symbol
-		(lib_id "Switch:SW_Push")
+		(lib_id "Keyboard Switches:SW_MX_HotSwap")
 		(at 148.59 66.04 0)
-		(mirror y)
 		(unit 1)
 		(exclude_from_sim no)
@@
 		(dnp no)
 		(property "Reference" "SW3"
-			(at 147.32 63.5 0)
+			(at 149.86 63.5 0)
 			(effects
 				(font
@@
 			)
 		)
-		(property "Footprint" ""
+		(property "Footprint" "Keyboard Switches:SW_MX_HotSwap"
 			(at 148.59 60.96 0)
 			(effects
@@
 	)
 	(symbol
-		(lib_id "Switch:SW_Push")
+		(lib_id "Keyboard Switches:SW_MX_HotSwap")
 		(at 148.59 76.2 0)
-		(mirror y)
 		(unit 1)
 		(exclude_from_sim no)
@@
 		(dnp no)
 		(property "Reference" "SW4"
-			(at 147.32 73.66 0)
+			(at 149.86 73.66 0)
 			(effects
 				(font
@@
 			)
 		)
-		(property "Footprint" ""
+		(property "Footprint" "Keyboard Switches:SW_MX_HotSwap"
 			(at 148.59 71.12 0)
 			(effects
